File: minime_2.1.1/minime_2.1.1.brd (EAGLE design)
At the start: 67 x 65.4 mm, 78 parts, among them J10 B2B-XH-A(LF)(SN), J12 B3B-XH-A(LF)(SN), J13 B2B-XH-A(LF)(SN), J14 B2B-XH-A(LF)(SN), J15 B4B-XH-AM(LF)(SN), J16 B3B-XH-A(LF)(SN), J6 B2B-XH-A(LF)(SN), J7 B2B-XH-A(LF)(SN), J8 B2B-XH-A(LF)(SN), J9 B2B-XH-A(LF)(SN)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

Commit message: minime_2.1.1
Parts:
- removed LED1: (no value), led:CHIP-LED0603
- removed R10, R9: 2k2, rcl:R0603
- added V1: NSI50010YT1GSOD, RPG_parts:SOD123
- C11, C12, C13: value (none) -> 22u
- R4: value 10k -> 680R
- R8: value 1k -> 0R
- moved U1 0.64 mm to (53.0, 45.4)
- moved R7 0.63 mm to (53.0, 48.3)
- moved LED5 0.45 mm to (50.5, 42.5), turned to 0 degrees
Connections:
- removed net N$32: LED1.A, R9.2
- removed net N$36: LED5.C, R10.2
- new net N$6: LED5.A, V1.C
- net +24V: no longer LED5.A
- net FAN2_STRG: no longer R9.1
- net GND: no longer LED1.C
- net N$35: now also LED5.C; no longer R10.1
- net N$41: now also V1.A
Routing:
- net +24V: track 221.1 -> 204.2 mm, vias 4 -> 2
- net N$41: track 17.4 -> 22.9 mm, vias 0 -> 1
- net N$6: track 0.00 -> 2.41 mm
- net N$35: track 12.3 -> 14.1 mm
- net N$36: track 1.42 -> 0.00 mm
- net N$32: track 1.36 -> 0.00 mm
Other:
- board text added: "by: kl33n 18.10.2021"
- board text removed: "by: kl33n 11.10.2021"
