File: minime_2.1.1/minime_2.1.1.sch (EAGLE design)
At the start: 78 parts, among them J10 B2B-XH-A(LF)(SN), J12 B3B-XH-A(LF)(SN), J13 B2B-XH-A(LF)(SN), J14 B2B-XH-A(LF)(SN), J15 B4B-XH-AM(LF)(SN), J16 B3B-XH-A(LF)(SN), J6 B2B-XH-A(LF)(SN), J7 B2B-XH-A(LF)(SN), J8 B2B-XH-A(LF)(SN), J9 B2B-XH-A(LF)(SN)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

Commit message: minime_2.1.1
Parts:
- removed LED1: (no value), led:LEDCHIP-LED0603
- removed R10, R9: 2k2, rcl:R-EU_R0603
- added V1: NSI50010YT1GSOD, RPG_parts:NSI50010YT1GSOD
- C11, C12, C13: value (none) -> 22u
- R4: value 10k -> 680R
- R8: value 1k -> 0R
Connections:
- removed net N$32: LED1.A, R9.2
- removed net N$36: LED5.C, R10.2
- new net N$6: LED5.A, V1.K
- net +24V: no longer LED5.A
- net FAN2_STRG: no longer R9.1
- net GND: no longer LED1.C
- net N$35: now also LED5.C; no longer R10.1
- net N$41: now also V1.A
Other:
- note added: "by: kl33n 18.10.2021"
- note removed: "by: kl33n 11.10.2021"
- moved on the sheet: LED5, R4
