File: minime_2.1.1/minime_2.1.1-a.brd (EAGLE design)
At the start: 67 x 65.4 mm, 76 parts, among them J10 B2B-XH-A(LF)(SN), J12 B3B-XH-A(LF)(SN), J13 B2B-XH-A(LF)(SN), J14 B2B-XH-A(LF)(SN), J15 B4B-XH-AM(LF)(SN), J16 B3B-XH-A(LF)(SN), J6 B2B-XH-A(LF)(SN), J7 B2B-XH-A(LF)(SN), J8 B2B-XH-A(LF)(SN), J9 B2B-XH-A(LF)(SN)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

Commit message: new version 2.1.1-a
Parts:
- removed J15: B4B-XH-AM(LF)(SN), B4B-XH-A:CONN_B4B-XH-AM_JST
- added J1: B2B-XH-A(LF)(SN), B2B-XH-A:CONN_B2B-XH-A(LF)(SN)_JST
- added LED1: (no value), led:CHIP-LED0603
- added R10: 10k, rcl:R0603
- added R9: 100R, rcl:R0603
- added U2: AO3400A, AO3400A:SOT-23-3L_AOS
- added V2: NSI50010YT1GSOD, RPG_parts:SOD123
- moved R11 0.63 mm to (53.0, 60.3)
- moved R21 0.63 mm to (26.7, 56.8)
- moved R12 0.32 mm to (51.4, 60.3)
- moved R22 0.32 mm to (28.3, 56.8)
Connections:
- new net N$12: J1.2, LED1.C, U2.3
- new net N$7: R10.2, R9.1, U2.1
- new net N$9: LED1.A, V2.C
- net FAN2_STRG: now also R9.2; no longer J15.2
- net GND: now also R10.1, U2.2; no longer J15.4
- net N$43: now also J1.1, V2.A; no longer J15.1
Routing:
- net N$12: track 0.00 -> 10.6 mm
- net FAN2_STRG: track 35.4 -> 27.2 mm
- net N$43: track 5.42 -> 10.6 mm
- net N$7: track 0.00 -> 3.88 mm
- net N$9: track 0.00 -> 3.77 mm
- net N$44: track 8.83 -> 9.99 mm
- net N$3: track 2.66 -> 3.29 mm
- net GND: track 59.6 -> 59.9 mm, vias 43 -> 49
Other:
- board text added: "F1"
- board text added: "F2"
- board text added: "by: kl33n 02.11.2021"
- board text added: "minime 2.1.1-a"
- board text removed: "by: kl33n 18.10.2021"
- board text removed: "minime 2.1.1"
