File: minime_2.1.1/minime_2.1.1-a.sch (EAGLE design)
At the start: 76 parts, among them J10 B2B-XH-A(LF)(SN), J12 B3B-XH-A(LF)(SN), J13 B2B-XH-A(LF)(SN), J14 B2B-XH-A(LF)(SN), J15 B4B-XH-AM(LF)(SN), J16 B3B-XH-A(LF)(SN), J6 B2B-XH-A(LF)(SN), J7 B2B-XH-A(LF)(SN), J8 B2B-XH-A(LF)(SN), J9 B2B-XH-A(LF)(SN)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

Commit message: new version 2.1.1-a
Parts:
- removed J15: B4B-XH-AM(LF)(SN), B4B-XH-A:B4B-XH-AM(LF)(SN)
- added J1: B2B-XH-A(LF)(SN), B2B-XH-A:B2B-XH-A(LF)(SN)
- added LED1: (no value), led:LEDCHIP-LED0603
- added R10: 10k, rcl:R-EU_R0603
- added R9: 100R, rcl:R-EU_R0603
- added U2: AO3400A, AO3400A:AO3400A
- added V2: NSI50010YT1GSOD, RPG_parts:NSI50010YT1GSOD
Connections:
- new net N$12: J1.2, LED1.C, U2.D
- new net N$7: R10.2, R9.1, U2.G
- new net N$9: LED1.A, V2.K
- net FAN2_STRG: now also R9.2; no longer J15.2
- net GND: now also R10.1, U2.S; no longer J15.4
- net N$43: now also J1.1, V2.A; no longer J15.1
Other:
- note added: "by: kl33n 02.11.2021"
- note added: "minime 2.1.1-a"
- note removed: "by: kl33n 18.10.2021"
- note removed: "minime 2.1.1"
- moved on the sheet: SJ4
